File: myProjects/2_Smart_Gateway/Hardware/V1.0/Smart_Gateway_V1.0/Smart_Gateway_V1.0.kicad_sch (KiCad schematic)
At the start: 57 parts, among them J1 USB_C_Receptacle_USB2.0_16P, J2 USB_C_Receptacle_USB2.0_16P, J3 Conn_01x06, J4 Conn_01x06, J5 Conn_01x06, Q1 BC847, Q2 BC847, SW1 CK_KMS2xxG, SW2 CK_KMS2xxG, SW3 CK_KMS2xxG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

Commit message: laptop
init
Parts:
- removed C10: 22uF/10V, Capacitor_SMD:C_0805_2012Metric, symbol Device:C
- removed C12, C13: 100nF/50V, Capacitor_SMD:C_0603_1608Metric, symbol Device:C
- removed C8: 100pF/16V, Capacitor_SMD:C_0603_1608Metric, symbol Device:C
- removed D10: WS2812B, LED_SMD:LED_WS2812B_PLCC4_5.0x5.0mm_P3.2mm, symbol LED:WS2812B
- removed D9: 1N4148W, Diode_SMD:D_SOD-123, symbol Diode:1N4148W
- removed L1: 1uH/3.2A, Inductor_SMD:L_APV_ANR252012, symbol Device:L
- removed R13: 10K, Resistor_SMD:R_0603_1608Metric, symbol Device:R
- removed R14: 100K, Resistor_SMD:R_0603_1608Metric, symbol Device:R
- removed R15: 22K, Resistor_SMD:R_0603_1608Metric, symbol Device:R
- removed R16: 3K3, Resistor_SMD:R_0603_1608Metric, symbol Device:R
- removed SW2, SW3: CK_KMS2xxG, Button_Switch_SMD:SW_SPST_CK_KMS2xxGP, symbol Switch:CK_KMS2xxG
- removed U2: TPS62A01PDDC, Package_TO_SOT_SMD:SOT-23-6, symbol Regulator_Switching:TPS62A01PDDC
- added D12, D13: LED, LED_SMD:LED_0603_1608Metric, symbol Device:LED
- added R20, R21: 3K3, Resistor_SMD:R_0603_1608Metric, symbol Device:R
- added U4: AMS1117-3.3, Package_TO_SOT_SMD:SOT-223-3_TabPin2, symbol Regulator_Linear:AMS1117-3.3
- J1, J2: footprint (none) -> Connector_USB:USB_C_Receptacle_GCT_USB4085
- J3, J4, J5: footprint SparkFun-Connector:1x06 -> Connector_PinSocket_2.54mm:PinSocket_1x06_P2.54mm_Vertical
- U3: footprint PCM_Espressif:ESP32-C6-WROOM-1 -> Esppressif:ESP32-C6-WROOM-1
Connections:
- net GPIO13 is gone; now on net GPIO12: D8.2 (A2), J2.A6 (D+), J2.B6 (D+), U3.14 (GPIO13/USB_D+)
- net +3.3V: now also U4.2 (VO)
- net +5.0V: now also U4.3 (VI)
- net Earth: now also J1.SH (SHIELD), J2.SH (SHIELD); no longer J1.S1 (SHIELD), J2.S1 (SHIELD)
- net GND: now also D12.1 (K), D13.1 (K), U4.1 (GND)
- net GPIO10: now also R21.1; no longer C11.1, SW1.2
- net GPIO11: now also C11.1, SW1.2
- net GPIO8: now also R20.1
- new net: D12.2 (A), R20.2
- new net: D13.2 (A), R21.2

Commit message: laptop
init
Other:
- moved on the sheet: R5, R6
Changed lines of the file:
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@@
 	)
 	(junction
-		(at 161.29 144.78)
+		(at 67.31 157.48)
 		(diameter 0)
 		(color 0 0 0 0)
 	)
 	(junction
-		(at 67.31 157.48)
+		(at 161.29 144.78)
 		(diameter 0)
 		(color 0 0 0 0)
@@
 	(wire
 		(pts
-			(xy 50.8 151.13) (xy 52.07 151.13)
+			(xy 50.8 151.13) (xy 54.61 151.13)
 		)
 		(stroke
@@
 	(wire
 		(pts
-			(xy 67.31 154.94) (xy 67.31 157.48)
+			(xy 67.31 148.59) (xy 67.31 157.48)
 		)
 		(stroke
@@
 	(wire
 		(pts
+			(xy 63.5 151.13) (xy 63.5 157.48)
+		)
+		(stroke
+			(width 0)
+			(type default)
+		)
+	)
+	(wire
+		(pts
 			(xy 59.69 161.29) (xy 59.69 162.56)
 		)
@@
 	(wire
 		(pts
-			(xy 220.98 110.49) (xy 220.98 104.14)
+			(xy 256.54 72.39) (xy 256.54 68.58)
 		)
 		(stroke
@@
 	(wire
 		(pts
-			(xy 173.99 154.94) (xy 198.12 154.94)
+			(xy 220.98 110.49) (xy 220.98 104.14)
 		)
 		(stroke
@@
 	(wire
 		(pts
-			(xy 347.98 160.02) (xy 358.14 160.02)
+			(xy 173.99 154.94) (xy 198.12 154.94)
 		)
 		(stroke
@@
 	(wire
 		(pts
-			(xy 234.95 139.7) (xy 248.92 139.7)
+			(xy 347.98 160.02) (xy 358.14 160.02)
 		)
 		(stroke
@@
 	(wire
 		(pts
-			(xy 347.98 142.24) (xy 358.14 142.24)
+			(xy 234.95 139.7) (xy 248.92 139.7)
 		)
 		(stroke
@@
 	(wire
 		(pts
-			(xy 332.74 217.17) (xy 337.82 217.17)
+			(xy 347.98 142.24) (xy 358.14 142.24)
 		)
 		(stroke
@@
 	(wire
 		(pts
-			(xy 185.42 149.86) (xy 198.12 149.86)
+			(xy 332.74 217.17) (xy 337.82 217.17)
 		)
 		(stroke
@@
 	(wire
 		(pts
-			(xy 53.34 154.94) (xy 54.61 154.94)
+			(xy 185.42 149.86) (xy 198.12 149.86)
 		)
 		(stroke
@@
 	(wire
 		(pts
-			(xy 62.23 157.48) (xy 67.31 157.48)
+			(xy 62.23 151.13) (xy 63.5 151.13)
 		)
 		(stroke
@@
 	(wire
 		(pts
-			(xy 52.07 157.48) (xy 54.61 157.48)
-		)
-		(stroke
-			(width 0)
-			(type default)
-		)
-	)
-	(wire
-		(pts
 			(xy 345.44 238.76) (xy 350.52 238.76)
 		)
@@
 	(wire
 		(pts
-			(xy 52.07 151.13) (xy 52.07 157.48)
-		)
-		(stroke
-			(width 0)
-			(type default)
-		)
-	)
-	(wire
-		(pts
 			(xy 50.8 161.29) (xy 59.69 161.29)
 		)
@@
 	(wire
 		(pts
-			(xy 53.34 148.59) (xy 53.34 154.94)
-		)
-		(stroke
-			(width 0)
-			(type default)
-		)
-	)
-	(wire
-		(pts
 			(xy 304.8 167.64) (xy 318.77 167.64)
 		)
@@
 	(wire
 		(pts
-			(xy 50.8 148.59) (xy 53.34 148.59)
+			(xy 50.8 148.59) (xy 54.61 148.59)
 		)
 		(stroke
@@
 	(wire
 		(pts
-			(xy 62.23 154.94) (xy 67.31 154.94)
+			(xy 62.23 148.59) (xy 67.31 148.59)
 		)
 		(stroke
@@
 	(wire
 		(pts
+			(xy 63.5 157.48) (xy 67.31 157.48)
+		)
+		(stroke
+			(width 0)
+			(type default)
+		)
+	)
+	(wire
+		(pts
 			(xy 49.53 102.87) (xy 58.42 102.87)
 		)
@@
 	(symbol
 		(lib_id "Device:R")
-		(at 58.42 157.48 90)
+		(at 58.42 151.13 90)
 		(mirror x)
 		(unit 1)
@@
 		(dnp no)
 		(property "Reference" "R6"
-			(at 55.88 159.512 90)
+			(at 55.88 153.162 90)
 			(show_name no)
 			(do_not_autoplace no)
@@
 		)
 		(property "Value" "5.1K"
-			(at 60.706 159.512 90)
+			(at 60.706 153.162 90)
 			(show_name no)
 			(do_not_autoplace no)
@@
 		)
 		(property "Footprint" "Resistor_SMD:R_0603_1608Metric"
-			(at 58.42 155.702 90)
+			(at 58.42 149.352 90)
 			(hide yes)
 			(show_name no)
@@
 		)
 		(property "Datasheet" ""
-			(at 58.42 157.48 0)
+			(at 58.42 151.13 0)
 			(hide yes)
 			(show_name no)
@@
 		)
 		(property "Description" ""
-			(at 58.42 157.48 0)
+			(at 58.42 151.13 0)
 			(hide yes)
 			(show_name no)
@@
 		)
 		(property "MP" ""
-			(at 58.42 157.48 90)
+			(at 58.42 151.13 90)
 			(hide yes)
 			(show_name no)
@@
 		)
 		(property "MF" ""
-			(at 58.42 157.48 90)
+			(at 58.42 151.13 90)
 			(hide yes)
 			(show_name no)
@@
 		)
 		(property "Package" "R0603"
-			(at 58.42 157.48 90)
+			(at 58.42 151.13 90)
 			(hide yes)
 			(show_name no)
@@
 	(symbol
 		(lib_id "power:GND")
-		(at 256.54 68.58 0)
+		(at 256.54 72.39 0)
 		(unit 1)
 		(body_style 1)
@@
 		(fields_autoplaced yes)
 		(property "Reference" "#PWR047"
-			(at 256.54 74.93 0)
+			(at 256.54 78.74 0)
 			(hide yes)
 			(show_name no)
@@
 		)
 		(property "Value" "GND"
-			(at 256.54 73.66 0)
+			(at 256.54 77.47 0)
 			(show_name no)
 			(do_not_autoplace no)
@@
 		)
 		(property "Footprint" ""
-			(at 256.54 68.58 0)
+			(at 256.54 72.39 0)
 			(hide yes)
 			(show_name no)
@@
 		)
 		(property "Datasheet" ""
-			(at 256.54 68.58 0)
+			(at 256.54 72.39 0)
 			(hide yes)
 			(show_name no)
@@
 		)
 		(property "Description" "Power symbol creates a global label with name \"GND\" , ground"
-			(at 256.54 68.58 0)
+			(at 256.54 72.39 0)
 			(hide yes)
 			(show_name no)
@@
 	(symbol
 		(lib_id "Device:R")
-		(at 58.42 154.94 90)
+		(at 58.42 148.59 90)
 		(unit 1)
 		(body_style 1)
@@
 		(dnp no)
 		(property "Reference" "R5"
-			(at 55.88 152.908 90)
+			(at 55.88 146.558 90)
 			(show_name no)
 			(do_not_autoplace no)
@@
 		)
 		(property "Value" "5.1K"
-			(at 60.706 152.908 90)
+			(at 60.706 146.558 90)
 			(show_name no)
 			(do_not_autoplace no)
@@
 		)
 		(property "Footprint" "Resistor_SMD:R_0603_1608Metric"
-			(at 58.42 156.718 90)
+			(at 58.42 150.368 90)
 			(hide yes)
 			(show_name no)
@@
 		)
 		(property "Datasheet" ""
-			(at 58.42 154.94 0)
+			(at 58.42 148.59 0)
 			(hide yes)
 			(show_name no)
@@
 		)
 		(property "Description" ""
-			(at 58.42 154.94 0)
+			(at 58.42 148.59 0)
 			(hide yes)
 			(show_name no)
@@
 		)
 		(property "MP" ""
-			(at 58.42 154.94 90)
+			(at 58.42 148.59 90)
 			(hide yes)
 			(show_name no)
@@
 		)
 		(property "MF" ""
-			(at 58.42 154.94 90)
+			(at 58.42 148.59 90)
 			(hide yes)
 			(show_name no)
@@
 		)
 		(property "Package" "R0603"
-			(at 58.42 154.94 90)
+			(at 58.42 148.59 90)
 			(hide yes)
 			(show_name no)
