File: myProjects/2_Smart_Gateway/Hardware/V1.0/Smart_Gateway_V1.0/Smart_Gateway_V1.0.kicad_pcb (KiCad board)
At the start: 2 copper layers, 44 x 44 mm, 0 parts

Commit message: laptop
init
Parts:
- added C1: 10uF/25V, Capacitor_SMD:C_0805_2012Metric, F.Cu at (158.2, 73.2)
- added C10: 22uF/10V, Capacitor_SMD:C_0805_2012Metric, F.Cu at (158.2, 88.3)
- added C11: 100nF/50V, Capacitor_SMD:C_0603_1608Metric, F.Cu at (162.5, 83.0)
- added C12: 100nF/50V, Capacitor_SMD:C_0603_1608Metric, F.Cu at (162.5, 85.5)
- added C13: 100nF/50V, Capacitor_SMD:C_0603_1608Metric, F.Cu at (162.5, 88.0)
- added C2: 10uF/25V, Capacitor_SMD:C_0805_2012Metric, F.Cu at (158.2, 76.2)
- added C3: 1uF/16V, Capacitor_SMD:C_0603_1608Metric, F.Cu at (162.5, 73.0)
- added C4: 4.7uF/25V, Capacitor_SMD:C_0805_2012Metric, F.Cu at (78.7, 82.3)
- added C4: 4.7uF/25V, Capacitor_SMD:C_0805_2012Metric, F.Cu at (158.2, 79.2)
- added C5: 10uF/25V, Capacitor_SMD:C_0805_2012Metric, F.Cu at (158.2, 82.3)
- added C6: 100nF/50V, Capacitor_SMD:C_0603_1608Metric, F.Cu at (162.5, 75.5)
- added C7: 1uF/16V, Capacitor_SMD:C_0603_1608Metric, F.Cu at (162.5, 78.0)
- added C8: 100pF/16V, Capacitor_SMD:C_0603_1608Metric, F.Cu at (162.5, 80.5)
- added C9: 22uF/10V, Capacitor_SMD:C_0805_2012Metric, F.Cu at (158.2, 85.3)
- added C9: 22uF/10V, Capacitor_SMD:C_0805_2012Metric, F.Cu at (78.7, 85.3)
- added D1: 5V, Diode_SMD:D_SOD-923, F.Cu at (198.5, 45.0)
- added D10: WS2812B, LED_SMD:LED_WS2812B_PLCC4_5.0x5.0mm_P3.2mm, F.Cu at (180.8, 85.8)
- added D11: LED, LED_SMD:LED_0603_1608Metric, F.Cu at (83.0, 82.1)
- added D11: LED, LED_SMD:LED_0603_1608Metric, F.Cu at (190.4, 70.6)
- added D12: LED, LED_SMD:LED_0603_1608Metric, F.Cu at (83.0, 84.7)
- added D13: LED, LED_SMD:LED_0603_1608Metric, F.Cu at (83.0, 87.3)
- added D2: 5V, Diode_SMD:D_SOD-923, F.Cu at (198.5, 46.9)
- added D3: 5V, Diode_SMD:D_SOD-923, F.Cu at (198.5, 48.9)
- added D4: 5V, Diode_SMD:D_SOD-923, F.Cu at (198.5, 50.8)
- added D5: 1N5819WS, Diode_SMD:D_SOD-323, F.Cu at (187.0, 84.0)
- added D6: 1N5819WS, Diode_SMD:D_SOD-323, F.Cu at (187.0, 86.9)
- added D7: 5V, Diode_SMD:D_SOD-923, F.Cu at (198.5, 52.8)
- added D8: 5V, Diode_SMD:D_SOD-923, F.Cu at (198.5, 54.7)
- added D9: 1N4148W, Diode_SMD:D_SOD-123, F.Cu at (191.2, 67.6)
- added J1: USB_C_Receptacle_USB2.0_16P, Connector_USB:USB_C_Receptacle_GCT_USB4085, F.Cu at (179.5, 62.9)
- added J2: USB_C_Receptacle_USB2.0_16P, Connector_USB:USB_C_Receptacle_GCT_USB4085, F.Cu at (183.3, 95.1)
- added J3: Conn_01x06, Connector_PinSocket_2.54mm:PinSocket_1x06_P2.54mm_Vertical, F.Cu at (218.8, 46.3)
- added J4: Conn_01x06, Connector_PinSocket_2.54mm:PinSocket_1x06_P2.54mm_Vertical, F.Cu at (223.4, 46.3)
- added J5: Conn_01x06, Connector_PinSocket_2.54mm:PinSocket_1x06_P2.54mm_Vertical, F.Cu at (228.0, 46.3)
- added L1: 1uH/3.2A, Inductor_SMD:L_APV_ANR252012, F.Cu at (195.5, 63.2)
- added Q1: BC847, Package_TO_SOT_SMD:SOT-23, F.Cu at (193.6, 74.7)
- added Q2: BC847, Package_TO_SOT_SMD:SOT-23, F.Cu at (193.6, 79.2)
- added R1: 1M, Resistor_SMD:R_0603_1608Metric, F.Cu at (166.5, 73.0)
- added R10: 470R, Resistor_SMD:R_0603_1608Metric, F.Cu at (170.5, 78.0)
- added R11: 10K, Resistor_SMD:R_0603_1608Metric, F.Cu at (170.5, 80.5)
- added R12: 10K, Resistor_SMD:R_0603_1608Metric, F.Cu at (170.5, 83.0)
- added R13: 10K, Resistor_SMD:R_0603_1608Metric, F.Cu at (170.5, 85.5)
- added R14: 100K, Resistor_SMD:R_0603_1608Metric, F.Cu at (170.5, 88.0)
- added R15: 22K, Resistor_SMD:R_0603_1608Metric, F.Cu at (174.5, 73.0)
- added R16: 3K3, Resistor_SMD:R_0603_1608Metric, F.Cu at (174.5, 75.5)
- added R17: 5.1K, Resistor_SMD:R_0603_1608Metric, F.Cu at (174.5, 78.0)
- added R17: 5.1K, Resistor_SMD:R_0603_1608Metric, F.Cu at (87.0, 82.1)
- added R18: 10K, Resistor_SMD:R_0603_1608Metric, F.Cu at (174.5, 80.5)
- added R19: 10K, Resistor_SMD:R_0603_1608Metric, F.Cu at (174.5, 83.0)
- added R2: 1M, Resistor_SMD:R_0603_1608Metric, F.Cu at (166.5, 75.5)
- added R20: 3K3, Resistor_SMD:R_0603_1608Metric, F.Cu at (87.0, 84.6)
- added R21: 3K3, Resistor_SMD:R_0603_1608Metric, F.Cu at (87.0, 87.1)
- added R3: 5.1K, Resistor_SMD:R_0603_1608Metric, F.Cu at (166.5, 78.0)
- added R4: 5.1K, Resistor_SMD:R_0603_1608Metric, F.Cu at (166.5, 80.5)
- added R5: 5.1K, Resistor_SMD:R_0603_1608Metric, F.Cu at (166.5, 83.0)
- added R6: 5.1K, Resistor_SMD:R_0603_1608Metric, F.Cu at (166.5, 85.5)
- added R7: 22.1K, Resistor_SMD:R_0603_1608Metric, F.Cu at (166.5, 88.0)
- added R8: 47.5K, Resistor_SMD:R_0603_1608Metric, F.Cu at (170.5, 73.0)
- added R9: 1K, Resistor_SMD:R_0603_1608Metric, F.Cu at (170.5, 75.5)
- added SW1: CK_KMS2xxG, Button_Switch_SMD:SW_SPST_CK_KMS2xxGP, F.Cu at (193.8, 46.5)
- added SW2: CK_KMS2xxG, Button_Switch_SMD:SW_SPST_CK_KMS2xxGP, F.Cu at (193.8, 51.9)
- added SW3: CK_KMS2xxG, Button_Switch_SMD:SW_SPST_CK_KMS2xxGP, F.Cu at (193.8, 57.3)
- added U1: CP2102N-Axx-xQFN28, Package_DFN_QFN:QFN-28-1EP_5x5mm_P0.5mm_EP3.35x3.35mm, F.Cu at (195.2, 85.0)
- added U2: TPS62A01PDDC, Package_TO_SOT_SMD:SOT-23-6, F.Cu at (190.9, 63.7)
- added U3: ESP32-C6-WROOM-1, Esppressif:ESP32-C6-WROOM-1, F.Cu at (175.0, 48.0)
- added U4: AMS1117-3.3, Package_TO_SOT_SMD:SOT-223-3_TabPin2, F.Cu at (81.4, 76.7)
Other:
- board size 44 x 44 mm -> 54.5 x 54.5 mm

Commit message: laptop
init
Parts:
- removed C10: 22uF/10V, Capacitor_SMD:C_0805_2012Metric
- removed C12, C13: 100nF/50V, Capacitor_SMD:C_0603_1608Metric
- removed the C4 at (78.7, 82.3)
- removed the C4 at (158.2, 79.2)
- removed C8: 100pF/16V, Capacitor_SMD:C_0603_1608Metric
- removed the C9 at (158.2, 85.3)
- removed the C9 at (78.7, 85.3)
- removed D10: WS2812B, LED_SMD:LED_WS2812B_PLCC4_5.0x5.0mm_P3.2mm
- removed the D11 at (83.0, 82.1)
- removed the D11 at (190.4, 70.6)
- removed D9: 1N4148W, Diode_SMD:D_SOD-123
- removed L1: 1uH/3.2A, Inductor_SMD:L_APV_ANR252012
- removed R13: 10K, Resistor_SMD:R_0603_1608Metric
- removed R14: 100K, Resistor_SMD:R_0603_1608Metric
- removed R15: 22K, Resistor_SMD:R_0603_1608Metric
- removed R16: 3K3, Resistor_SMD:R_0603_1608Metric
- removed the R17 at (174.5, 78.0)
- removed the R17 at (87.0, 82.1)
- removed SW2, SW3: CK_KMS2xxG, Button_Switch_SMD:SW_SPST_CK_KMS2xxGP
- removed U2: TPS62A01PDDC, Package_TO_SOT_SMD:SOT-23-6
- removed U3: ESP32-C6-WROOM-1, Esppressif:ESP32-C6-WROOM-1
- added C4: 4.7uF/25V, Capacitor_SMD:C_0805_2012Metric, F.Cu at (215.4, 143.5)
- added C9: 22uF/10V, Capacitor_SMD:C_0805_2012Metric, F.Cu at (215.4, 149.5)
- added D11: LED, LED_SMD:LED_0603_1608Metric, F.Cu at (218.4, 128.0)
- added R17: 5.1K, Resistor_SMD:R_0603_1608Metric, F.Cu at (209.5, 124.7)
- moved D12 143.0 mm to (218.4, 130.6)
- moved D13 143.0 mm to (218.4, 133.2)
- moved U4 142.6 mm to (216.4, 122.6)
- moved R20 131.4 mm to (209.5, 132.2)
- moved R21 131.4 mm to (209.5, 134.7)
- moved SW1 104.1 mm to (191.1, 150.6)
- moved D2 94.3 mm to (219.1, 138.9)
- moved D1 94.3 mm to (219.1, 136.9)
- moved D3 94.3 mm to (219.1, 140.8)
- moved D7 94.3 mm to (219.1, 144.7)
- moved D8 94.3 mm to (219.1, 146.7)
- moved D4 94.3 mm to (219.1, 142.8)
- moved J3 93.5 mm to (201.7, 138.3)
- moved J4 93.5 mm to (206.3, 138.3)
- moved J5 93.5 mm to (210.9, 138.3)
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Other:
- outline, holes or cut-outs redrawn

Commit message: PC
İNİT
Parts:
- removed C1, C2, C5: 10uF/25V, Capacitor_SMD:C_0805_2012Metric
- removed C11, C6: 100nF/50V, Capacitor_SMD:C_0603_1608Metric
- removed C3, C7: 1uF/16V, Capacitor_SMD:C_0603_1608Metric
- removed C4: 4.7uF/25V, Capacitor_SMD:C_0805_2012Metric
- removed C9: 22uF/10V, Capacitor_SMD:C_0805_2012Metric
- removed D1, D2, D3, D4, D7, D8: 5V, Diode_SMD:D_SOD-923
- removed D11, D12, D13: LED, LED_SMD:LED_0603_1608Metric
- removed D5, D6: 1N5819WS, Diode_SMD:D_SOD-323
- removed J1, J2: USB_C_Receptacle_USB2.0_16P, Connector_USB:USB_C_Receptacle_GCT_USB4085
- removed J3, J4, J5: Conn_01x06, Connector_PinSocket_2.54mm:PinSocket_1x06_P2.54mm_Vertical
- removed Q1, Q2: BC847, Package_TO_SOT_SMD:SOT-23
- removed R1, R2: 1M, Resistor_SMD:R_0603_1608Metric
- removed R10: 470R, Resistor_SMD:R_0603_1608Metric
- removed R11, R12, R18, R19: 10K, Resistor_SMD:R_0603_1608Metric
- removed R17, R3, R4, R5, R6: 5.1K, Resistor_SMD:R_0603_1608Metric
- removed R20, R21: 3K3, Resistor_SMD:R_0603_1608Metric
- removed R7: 22.1K, Resistor_SMD:R_0603_1608Metric
- removed R8: 47.5K, Resistor_SMD:R_0603_1608Metric
- removed R9: 1K, Resistor_SMD:R_0603_1608Metric
- removed SW1: CK_KMS2xxG, Button_Switch_SMD:SW_SPST_CK_KMS2xxGP
- removed U1: CP2102N-Axx-xQFN28, Package_DFN_QFN:QFN-28-1EP_5x5mm_P0.5mm_EP3.35x3.35mm
- removed U4: AMS1117-3.3, Package_TO_SOT_SMD:SOT-223-3_TabPin2
Other:
- board size 54.5 x 54.5 mm -> 55 x 55 mm
- rule pad_to_mask_clearance: 0 -> 0.1016
